Commit message: feat: add collisions and inertia to robot urdf

File: src/sgm_robot_description/urdf/sgm_robot.urdf.xacro (robot description, xacro)
@@ -16,5 +16,35 @@
     <xacro:property name="camera_height" value="0.05" />
     <xacro:property name="laser_radius" value="0.1" />
-    <xacro:property name="laser_height" value="0.01" />
+    <xacro:property name="laser_height" value="0.03" />
+    <!-- inertias -->
+    <!-- http://wiki.ros.org/urdf/Tutorials/Adding%20Physical%20and%20Collision%20Properties%20to%20a%20URDF%20Model -->
+    <xacro:macro name="box_inertia" params="m l w h xyz rpy">
+        <inertial>
+            <origin xyz="${xyz}" rpy="${rpy}" />
+            <mass value="${m}" />
+            <inertia ixx="${(m/12) * (h*h + l*l)}" ixy="0" ixz="0"
+                     iyy="${(m/12) * (w*w + l*l)}" iyz="0"
+                     izz="${(m/12) * (w*w + h*h)}" />
+        </inertial>
+    </xacro:macro>
+    <xacro:macro name="cylinder_inertia" params="m r h xyz rpy">
+        <inertial>
+            <origin xyz="${xyz}" rpy="${rpy}" />
+            <mass value="${m}" />
+            <inertia ixx="${(m/12) * (3*r*r + h*h)}" ixy="0" ixz="0"
+                     iyy="${(m/12) * (3*r*r + h*h)}" iyz="0"
+                     izz="${(m/2) * (r*r)}" />
+        </inertial>
+    </xacro:macro>
+    <xacro:macro name="sphere_inertia" params="m r xyz rpy">
+        <inertial>
+            <origin xyz="${xyz}" rpy="${rpy}" />
+            <mass value="${m}" />
+            <inertia ixx="${(2/5) * m * r * r}" ixy="0" ixz="0"
+                     iyy="${(2/5) * m * r * r}" iyz="0"
+                     izz="${(2/5) * m * r * r}" />
+        </inertial>
+    </xacro:macro>
+    <!-- base -->
 	<link name="base_footprint" />
 	<link name="base_link">
@@ -23,7 +53,15 @@
 				<box size="${base_length} ${base_width} ${base_height}" />
 			</geometry>
-			<origin xyz="0 0 ${wheel_radius}" rpy="0 0 0" />
+			<origin xyz="0 0 ${base_height / 2.0}" rpy="0 0 0" />
 			<material name="dark_grey" />
 		</visual>
+        <collision>
+            <geometry>
+                <box size="${base_length} ${base_width} ${base_height}" />
+            </geometry>
+            <origin xyz="0 0 ${base_height / 2.0}" rpy="0 0 0" />
+        </collision>
+        <xacro:box_inertia m="5.0" l="${2*base_length}" w="${2*base_width}" h="${2*base_height}"
+                           xyz="0 0 ${base_height / 2.0}" rpy="0 0 0" />
 	</link>
     <joint name="base_joint" type="fixed">
@@ -42,4 +80,12 @@
                 <material name="light_grey" />
             </visual>
+            <collision>
+                <geometry>
+                    <cylinder radius="${wheel_radius}" length="${wheel_width}" />
+                </geometry>
+                <origin xyz="0 0 0" rpy="${pi / 2.0} 0 0" />
+            </collision>
+            <xacro:cylinder_inertia m="1.0" r="${2*wheel_radius}" h="${2*wheel_width}"
+                                    xyz="0 0 0" rpy="${pi / 2.0} 0 0" />
         </link>
     </xacro:macro>
@@ -54,4 +100,12 @@
             <material name="light_grey" />
         </visual>
+        <collision>
+            <geometry>
+                <sphere radius="${wheel_radius / 2.0}" />
+            </geometry>
+            <origin xyz="0 0 0" rpy="0 0 0" />
+        </collision>
+        <xacro:sphere_inertia m="0.5" r="${2*wheel_radius / 2.0}"
+                              xyz="0 0 0" rpy="0 0 0" />
     </link>
     <joint name="base_right_wheel_joint" type="continuous">
@@ -80,4 +134,11 @@
             <material name="light_grey" />
         </visual>
+        <collision>
+            <geometry>
+                <box size="${camera_length} ${camera_width} ${camera_height}" />
+            </geometry>
+        </collision>
+        <xacro:box_inertia m="0.1" l="${camera_length}" w="${camera_width}" h="${camera_height}"
+                           xyz="0 0 0" rpy="0 0 0" />
     </link>
     <joint name="base_camera_joint" type="fixed">
@@ -94,4 +155,11 @@
             <material name="light_grey" />
         </visual>
+        <collision>
+            <geometry>
+                <cylinder radius="${laser_radius}" length="${laser_height}" />
+            </geometry>
+        </collision>
+        <xacro:cylinder_inertia m="1.0" r="${2*laser_radius}" h="${2*laser_height}"
+                                xyz="0 0 0" rpy="0 0 0" />
     </link>
     <joint name="base_laser_joint" type="fixed">

Commit message: feat: add gazebo colors to robot

File: src/sgm_robot_description/urdf/sgm_robot.urdf.xacro (robot description, xacro)
@@ -168,4 +168,24 @@
         <origin xyz="${base_length / 8} 0 ${base_height}" rpy="0 0 0" />
     </joint>
+    <gazebo reference="base_link">
+        <material>Gazebo/Blue</material>
+    </gazebo>
+    <gazebo reference="right_wheel_link">
+        <material>Gazebo/Grey</material>
+    </gazebo>
+    <gazebo reference="left_wheel_link">
+        <material>Gazebo/Grey</material>
+    </gazebo>
+    <gazebo reference="caster_wheel_link">
+        <material>Gazebo/Grey</material>
+        <mu1 value="0.1" />
+        <mu2 value="0.1" />
+    </gazebo>
+    <gazebo reference="laser_link">
+        <material>Gazebo/Grey</material>
+    </gazebo>
+    <gazebo reference="camera_link">
+        <material>Gazebo/Grey</material>
+    </gazebo>
     <gazebo>
         <plugin name="diff_drive_controller" filename="libgazebo_ros_diff_drive.so">

Commit message: feat: add camera plugin to robot

File: src/sgm_robot_description/urdf/sgm_robot.urdf.xacro (robot description, xacro)
@@ -186,5 +186,5 @@
     </gazebo>
     <gazebo reference="camera_link">
-        <material>Gazebo/Grey</material>
+        <material>Gazebo/Red</material>
     </gazebo>
     <gazebo>
@@ -203,3 +203,20 @@
         </plugin>
     </gazebo>
+    <link name="camera_link_optical" />
+    <joint name="camera_optical_joint" type="fixed">
+        <origin xyz="0 0 0" rpy="${-pi/2} 0 ${-pi/2}"/>
+        <parent link="camera_link"/>
+        <child link="camera_link_optical"/>
+    </joint>
+    <gazebo reference="camera_link">
+        <material>Gazebo/Red</material>
+        <sensor name="camera_sensor" type="camera">
+            <pose>0 0 0 0 0 0</pose>
+            <visualize>true</visualize>
+            <update_rate>10.0</update_rate>
+            <plugin name="camera_controller" filename="libgazebo_ros_camera.so">
+                <frame_name>camera_link_optical</frame_name>
+            </plugin>
+        </sensor>
+    </gazebo>
 </robot>

Commit message: feat: add laserscan plugin to robot

File: src/sgm_robot_description/urdf/sgm_robot.urdf.xacro (robot description, xacro)
@@ -16,5 +16,5 @@
     <xacro:property name="camera_height" value="0.05" />
     <xacro:property name="laser_radius" value="0.1" />
-    <xacro:property name="laser_height" value="0.03" />
+    <xacro:property name="laser_height" value="0.06" />
     <!-- inertias -->
     <!-- http://wiki.ros.org/urdf/Tutorials/Adding%20Physical%20and%20Collision%20Properties%20to%20a%20URDF%20Model -->
@@ -183,5 +183,5 @@
     </gazebo>
     <gazebo reference="laser_link">
-        <material>Gazebo/Grey</material>
+        <material>Gazebo/Red</material>
     </gazebo>
     <gazebo reference="camera_link">
@@ -220,3 +220,37 @@
         </sensor>
     </gazebo>
+    <link name="laser_link_scan" />
+    <joint name="laser_scan_joint" type="fixed">
+        <origin xyz="0 0 ${(laser_height/2) + 0.05}" rpy="0 0 0"/>
+        <parent link="laser_link"/>
+        <child link="laser_link_scan"/>
+    </joint>
+    <gazebo reference="laser_link_scan">
+        <material>Gazebo/Red</material>
+        <sensor name="laser" type="ray">
+            <pose> 0 0 0 0 0 0 </pose>
+            <visualize>true</visualize>
+            <update_rate>10</update_rate>
+            <ray>
+                <scan>
+                    <horizontal>
+                        <samples>360</samples>
+                        <min_angle>-3.14</min_angle>
+                        <max_angle>3.14</max_angle>
+                    </horizontal>
+                </scan>
+                <range>
+                    <min>0.3</min>
+                    <max>12</max>
+                </range>
+            </ray>
+            <plugin name="laser_controller" filename="libgazebo_ros_ray_sensor.so">
+                <ros>
+                    <argument>~/out:=scan</argument>
+                </ros>
+                <output_type>sensor_msgs/LaserScan</output_type>
+                <frame_name>laser_link_scan</frame_name>
+            </plugin>
+        </sensor>
+    </gazebo>
 </robot>

Commit message: update: give no friction to robot

File: src/sgm_robot_description/urdf/sgm_robot.urdf.xacro (robot description, xacro)
@@ -1,10 +1,11 @@
 <?xml version="1.0"?>
-<robot name="sgm_robot" xmlns:xacro="http://www.ros.org/wiki/xacro">
-	<material name="dark_grey">
-		<color rgba="0.2 0.2 0.2 1"></color>
-	</material>
-	<material name="light_grey">
-		<color rgba="0.8 0.8 0.8 1"></color>
-	</material>
+<robot name="sgm_robot"
+    xmlns:xacro="http://www.ros.org/wiki/xacro">
+    <material name="dark_grey">
+        <color rgba="0.2 0.2 0.2 1"></color>
+    </material>
+    <material name="light_grey">
+        <color rgba="0.8 0.8 0.8 1"></color>
+    </material>
     <xacro:property name="base_length" value="0.6" />
     <xacro:property name="base_width" value="0.4" />
@@ -23,7 +24,5 @@
             <origin xyz="${xyz}" rpy="${rpy}" />
             <mass value="${m}" />
-            <inertia ixx="${(m/12) * (h*h + l*l)}" ixy="0" ixz="0"
-                     iyy="${(m/12) * (w*w + l*l)}" iyz="0"
-                     izz="${(m/12) * (w*w + h*h)}" />
+            <inertia ixx="${(m/12) * (h*h + l*l)}" ixy="0" ixz="0" iyy="${(m/12) * (w*w + l*l)}" iyz="0" izz="${(m/12) * (w*w + h*h)}" />
         </inertial>
     </xacro:macro>
@@ -32,7 +31,5 @@
             <origin xyz="${xyz}" rpy="${rpy}" />
             <mass value="${m}" />
-            <inertia ixx="${(m/12) * (3*r*r + h*h)}" ixy="0" ixz="0"
-                     iyy="${(m/12) * (3*r*r + h*h)}" iyz="0"
-                     izz="${(m/2) * (r*r)}" />
+            <inertia ixx="${(m/12) * (3*r*r + h*h)}" ixy="0" ixz="0" iyy="${(m/12) * (3*r*r + h*h)}" iyz="0" izz="${(m/2) * (r*r)}" />
         </inertial>
     </xacro:macro>
@@ -41,33 +38,30 @@
             <origin xyz="${xyz}" rpy="${rpy}" />
             <mass value="${m}" />
-            <inertia ixx="${(2/5) * m * r * r}" ixy="0" ixz="0"
-                     iyy="${(2/5) * m * r * r}" iyz="0"
-                     izz="${(2/5) * m * r * r}" />
+            <inertia ixx="${(2/5) * m * r * r}" ixy="0" ixz="0" iyy="${(2/5) * m * r * r}" iyz="0" izz="${(2/5) * m * r * r}" />
         </inertial>
     </xacro:macro>
     <!-- base -->
-	<link name="base_footprint" />
-	<link name="base_link">
-		<visual>
-			<geometry>
-				<box size="${base_length} ${base_width} ${base_height}" />
-			</geometry>
-			<origin xyz="0 0 ${base_height / 2.0}" rpy="0 0 0" />
-			<material name="dark_grey" />
-		</visual>
-        <collision>
+    <link name="base_footprint" />
+    <link name="base_link">
+        <visual>
             <geometry>
                 <box size="${base_length} ${base_width} ${base_height}" />
             </geometry>
             <origin xyz="0 0 ${base_height / 2.0}" rpy="0 0 0" />
-        </collision>
-        <xacro:box_inertia m="5.0" l="${2*base_length}" w="${2*base_width}" h="${2*base_height}"
-                           xyz="0 0 ${base_height / 2.0}" rpy="0 0 0" />
-	</link>
+            <material name="dark_grey" />
+        </visual>
+        <collision>
+            <geometry>
+                <box size="${base_length} ${base_width} ${base_height}" />
+            </geometry>
+            <origin xyz="0 0 ${base_height / 2.0}" rpy="0 0 0" />
+        </collision>
+        <xacro:box_inertia m="5.0" l="${2*base_length}" w="${2*base_width}" h="${2*base_height}" xyz="0 0 ${base_height / 2.0}" rpy="0 0 0" />
+    </link>
     <joint name="base_joint" type="fixed">
-		<parent link="base_footprint" />
-		<child link="base_link" />
-		<origin xyz="0 0 ${wheel_radius}" rpy="0 0 0"/>
-	</joint>
+        <parent link="base_footprint" />
+        <child link="base_link" />
+        <origin xyz="0 0 ${wheel_radius}" rpy="0 0 0"/>
+    </joint>
     <!-- wheels -->
     <xacro:macro name="wheel_link" params="prefix">
@@ -86,6 +80,5 @@
                 <origin xyz="0 0 0" rpy="${pi / 2.0} 0 0" />
             </collision>
-            <xacro:cylinder_inertia m="1.0" r="${2*wheel_radius}" h="${2*wheel_width}"
-                                    xyz="0 0 0" rpy="${pi / 2.0} 0 0" />
+            <xacro:cylinder_inertia m="1.0" r="${2*wheel_radius}" h="${2*wheel_width}" xyz="0 0 0" rpy="${pi / 2.0} 0 0" />
         </link>
     </xacro:macro>
@@ -106,6 +99,5 @@
             <origin xyz="0 0 0" rpy="0 0 0" />
         </collision>
-        <xacro:sphere_inertia m="0.5" r="${2*wheel_radius / 2.0}"
-                              xyz="0 0 0" rpy="0 0 0" />
+        <xacro:sphere_inertia m="0.5" r="${2*wheel_radius / 2.0}" xyz="0 0 0" rpy="0 0 0" />
     </link>
     <joint name="base_right_wheel_joint" type="continuous">
@@ -139,6 +131,5 @@
             </geometry>
         </collision>
-        <xacro:box_inertia m="0.1" l="${camera_length}" w="${camera_width}" h="${camera_height}"
-                           xyz="0 0 0" rpy="0 0 0" />
+        <xacro:box_inertia m="0.1" l="${camera_length}" w="${camera_width}" h="${camera_height}" xyz="0 0 0" rpy="0 0 0" />
     </link>
     <joint name="base_camera_joint" type="fixed">
@@ -160,6 +151,5 @@
             </geometry>
         </collision>
-        <xacro:cylinder_inertia m="1.0" r="${2*laser_radius}" h="${2*laser_height}"
-                                xyz="0 0 0" rpy="0 0 0" />
+        <xacro:cylinder_inertia m="1.0" r="${2*laser_radius}" h="${2*laser_height}" xyz="0 0 0" rpy="0 0 0" />
     </link>
     <joint name="base_laser_joint" type="fixed">
@@ -173,12 +163,16 @@
     <gazebo reference="right_wheel_link">
         <material>Gazebo/Grey</material>
+        <mu1 value="0.0"/>
+        <mu2 value="0.0"/>
     </gazebo>
     <gazebo reference="left_wheel_link">
         <material>Gazebo/Grey</material>
+        <mu1 value="0.0"/>
+        <mu2 value="0.0"/>
     </gazebo>
     <gazebo reference="caster_wheel_link">
         <material>Gazebo/Grey</material>
-        <mu1 value="0.1" />
-        <mu2 value="0.1" />
+        <mu1 value="0.0" />
+        <mu2 value="0.0" />
     </gazebo>
     <gazebo reference="laser_link">
